File: ATF1502AS-EVB/ATF1502AS-EVB.sch (KiCad schematic (older format))
At the start: 16 parts, among them J1 Conn_02x03_Odd_Even, J2 Conn_01x20, J3 Conn_01x20, U1 ATF1502AS

Commit message: Update for upstream changes.
Parts:
- J2, J3: footprint Connector_PinHeader_2.54mm:PinHeader_1x20_P2.54mm_Vertical -> ATF1502AS-EVB:PinSocket_1x20_P2.54mm_Vertical_NoSilk
- U1: value ATF1502AS -> ATF1502AS-xAx44; symbol CPLD_Microchip:ATF1502AS -> CPLD_Microchip:ATF1502AS-xAx44
Changed lines of the file:
@@
 $EndDescr
-$Comp
-L CPLD_Microchip:ATF1502AS U1
-U 1 1 5DF180CF
-P 2600 4250
-F 0 "U1" H 2150 5200 50  0000 C CNN
-F 1 "ATF1502AS" H 2900 5200 50  0000 C CNN
-F 2 "Package_QFP:TQFP-44_10x10mm_P0.8mm" H 2600 5800 50  0001 C CNN
-F 3 "http://ww1.microchip.com/downloads/en/DeviceDoc/Atmel-0995-CPLD-ATF1502AS(L)-Datasheet.pdf" H 2600 5700 50  0001 C CNN
-	1    2600 4250
-	1    0    0    -1
-$EndComp
 $Comp
 L Connector_Generic:Conn_01x20 J2
@@
 F 0 "J2" H 1450 3150 50  0000 C CNN
 F 1 "Conn_01x20" H 1368 3116 50  0001 C CNN
-F 2 "Connector_PinHeader_2.54mm:PinHeader_1x20_P2.54mm_Vertical" H 1450 4250 50  0001 C CNN
+F 2 "ATF1502AS-EVB:PinSocket_1x20_P2.54mm_Vertical_NoSilk" H 1450 4250 50  0001 C CNN
 F 3 "~" H 1450 4250 50  0001 C CNN
 	1    1450 4250
@@
 F 0 "J3" H 3750 5150 50  0000 C CNN
 F 1 "Conn_01x20" H 3668 5176 50  0001 C CNN
-F 2 "Connector_PinHeader_2.54mm:PinHeader_1x20_P2.54mm_Vertical" H 3750 4150 50  0001 C CNN
+F 2 "ATF1502AS-EVB:PinSocket_1x20_P2.54mm_Vertical_NoSilk" H 3750 4150 50  0001 C CNN
 F 3 "~" H 3750 4150 50  0001 C CNN
 	1    3750 4150
@@
 Wire Wire Line
 	5050 3650 5050 3700
+$Comp
+L CPLD_Microchip:ATF1502AS-xAx44 U1
+U 1 1 5DF180CF
+P 2600 4250
+F 0 "U1" H 2150 5200 50  0000 C CNN
+F 1 "ATF1502AS-xAx44" H 2200 3200 50  0000 C CNN
+F 2 "Package_QFP:TQFP-44_10x10mm_P0.8mm" H 2600 5800 50  0001 C CNN
+F 3 "http://ww1.microchip.com/downloads/en/DeviceDoc/Atmel-0995-CPLD-ATF1502AS(L)-Datasheet.pdf" H 2600 5700 50  0001 C CNN
+	1    2600 4250
+	1    0    0    -1
+$EndComp
 $EndSCHEMATC

Commit message: ATF1502AS-EVB: final changes for fab.
Parts:
- D1, D2, D3: value LED -> GRN; MPN (none) -> 150060GS75000; Mfg (none) -> Wurth
- J1: value Conn_02x03_Odd_Even -> VERT
- J2, J3: value Conn_01x20 -> VERT; footprint ATF1502AS-EVB:PinSocket_1x20_P2.54mm_Vertical_NoSilk -> ATF1502AS-EVB:PinHeader_1x20_P2.54mm_Vertical_NoSilk
- JP1, JP2: value SolderJumper_2_Open -> DNP
- R1, R2, R3: value 3k3 -> 10k
- U1: MPN (none) -> ATF1502AS-7AX44; Mfg (none) -> Microchip
Changed lines of the file:
@@
 P 1450 4250
 F 0 "J2" H 1450 3150 50  0000 C CNN
-F 1 "Conn_01x20" H 1368 3116 50  0001 C CNN
-F 2 "ATF1502AS-EVB:PinSocket_1x20_P2.54mm_Vertical_NoSilk" H 1450 4250 50  0001 C CNN
+F 1 "VERT" H 1368 3116 50  0001 C CNN
+F 2 "ATF1502AS-EVB:PinHeader_1x20_P2.54mm_Vertical_NoSilk" H 1450 4250 50  0001 C CNN
 F 3 "~" H 1450 4250 50  0001 C CNN
 	1    1450 4250
@@
 P 3750 4150
 F 0 "J3" H 3750 5150 50  0000 C CNN
-F 1 "Conn_01x20" H 3668 5176 50  0001 C CNN
-F 2 "ATF1502AS-EVB:PinSocket_1x20_P2.54mm_Vertical_NoSilk" H 3750 4150 50  0001 C CNN
+F 1 "VERT" H 3668 5176 50  0001 C CNN
+F 2 "ATF1502AS-EVB:PinHeader_1x20_P2.54mm_Vertical_NoSilk" H 3750 4150 50  0001 C CNN
 F 3 "~" H 3750 4150 50  0001 C CNN
 	1    3750 4150
@@
 P 4700 2450
 F 0 "J1" H 4750 2675 50  0000 C CNN
-F 1 "Conn_02x03_Odd_Even" H 4750 2676 50  0001 C CNN
+F 1 "VERT" H 4750 2676 50  0001 C CNN
 F 2 "Connector_PinHeader_2.54mm:PinHeader_2x03_P2.54mm_Vertical" H 4700 2450 50  0001 C CNN
 F 3 "~" H 4700 2450 50  0001 C CNN
@@
 P 4450 3850
 F 0 "R1" H 4520 3896 50  0000 L CNN
-F 1 "3k3" H 4520 3805 50  0000 L CNN
+F 1 "10k" H 4520 3805 50  0000 L CNN
 F 2 "Resistor_SMD:R_0805_2012Metric_Pad1.15x1.40mm_HandSolder" V 4380 3850 50  0001 C CNN
 F 3 "~" H 4450 3850 50  0001 C CNN
@@
 P 4750 3850
 F 0 "R3" H 4820 3896 50  0000 L CNN
-F 1 "3k3" H 4820 3805 50  0000 L CNN
+F 1 "10k" H 4820 3805 50  0000 L CNN
 F 2 "Resistor_SMD:R_0805_2012Metric_Pad1.15x1.40mm_HandSolder" V 4680 3850 50  0001 C CNN
 F 3 "~" H 4750 3850 50  0001 C CNN
@@
 P 5050 3850
 F 0 "R2" H 5120 3896 50  0000 L CNN
-F 1 "3k3" H 5120 3805 50  0000 L CNN
+F 1 "10k" H 5120 3805 50  0000 L CNN
 F 2 "Resistor_SMD:R_0805_2012Metric_Pad1.15x1.40mm_HandSolder" V 4980 3850 50  0001 C CNN
 F 3 "~" H 5050 3850 50  0001 C CNN
 	1    5050 3850
 	1    0    0    -1
-$EndComp
-$Comp
-L Device:LED D1
-U 1 1 5DF6B205
-P 4450 4200
-F 0 "D1" V 4450 4150 50  0000 R CNN
-F 1 "LED" V 4398 4083 50  0001 R CNN
-F 2 "LED_SMD:LED_0603_1608Metric_Pad1.05x0.95mm_HandSolder" H 4450 4200 50  0001 C CNN
-F 3 "~" H 4450 4200 50  0001 C CNN
-	1    4450 4200
-	0    -1   -1   0
-$EndComp
-$Comp
-L Device:LED D3
-U 1 1 5DF6CDCD
-P 4750 4200
-F 0 "D3" V 4750 4150 50  0000 R CNN
-F 1 "LED" V 4698 4083 50  0001 R CNN
-F 2 "LED_SMD:LED_0603_1608Metric_Pad1.05x0.95mm_HandSolder" H 4750 4200 50  0001 C CNN
-F 3 "~" H 4750 4200 50  0001 C CNN
-	1    4750 4200
-	0    -1   -1   0
-$EndComp
-$Comp
-L Device:LED D2
-U 1 1 5DF6D134
-P 5050 4200
-F 0 "D2" V 5050 4150 50  0000 R CNN
-F 1 "LED" V 4998 4083 50  0001 R CNN
-F 2 "LED_SMD:LED_0603_1608Metric_Pad1.05x0.95mm_HandSolder" H 5050 4200 50  0001 C CNN
-F 3 "~" H 5050 4200 50  0001 C CNN
-	1    5050 4200
-	0    -1   -1   0
 $EndComp
 Wire Wire Line
@@
 P 4450 3500
 F 0 "JP1" V 4450 3568 50  0000 L CNN
-F 1 "SolderJumper_2_Open" V 4495 3568 50  0001 L CNN
+F 1 "DNP" V 4495 3568 50  0001 L CNN
 F 2 "Jumper:SolderJumper-2_P1.3mm_Open_TrianglePad1.0x1.5mm" H 4450 3500 50  0001 C CNN
 F 3 "~" H 4450 3500 50  0001 C CNN
@@
 P 5050 3500
 F 0 "JP2" V 5050 3568 50  0000 L CNN
-F 1 "SolderJumper_2_Open" V 5095 3568 50  0001 L CNN
+F 1 "DNP" V 5095 3568 50  0001 L CNN
 F 2 "Jumper:SolderJumper-2_P1.3mm_Open_TrianglePad1.0x1.5mm" H 5050 3500 50  0001 C CNN
 F 3 "~" H 5050 3500 50  0001 C CNN
@@
 F 2 "Package_QFP:TQFP-44_10x10mm_P0.8mm" H 2600 5800 50  0001 C CNN
 F 3 "http://ww1.microchip.com/downloads/en/DeviceDoc/Atmel-0995-CPLD-ATF1502AS(L)-Datasheet.pdf" H 2600 5700 50  0001 C CNN
+F 4 "ATF1502AS-7AX44" H 2600 4250 50  0001 C CNN "MPN"
+F 5 "Microchip" H 2600 4250 50  0001 C CNN "Mfg"
 	1    2600 4250
 	1    0    0    -1
 $EndComp
+$Comp
+L Device:LED D2
+U 1 1 5DF6D134
+P 5050 4200
+F 0 "D2" V 5050 4150 50  0000 R CNN
+F 1 "GRN" V 4900 4100 50  0000 R CNN
+F 2 "LED_SMD:LED_0603_1608Metric_Pad1.05x0.95mm_HandSolder" H 5050 4200 50  0001 C CNN
+F 3 "~" H 5050 4200 50  0001 C CNN
+F 4 "150060GS75000" H 5050 4200 50  0001 C CNN "MPN"
+F 5 "Wurth" H 5050 4200 50  0001 C CNN "Mfg"
+	1    5050 4200
+	0    -1   -1   0
+$EndComp
+$Comp
+L Device:LED D3
+U 1 1 5DF6CDCD
+P 4750 4200
+F 0 "D3" V 4750 4150 50  0000 R CNN
+F 1 "GRN" V 4600 4100 50  0000 R CNN
+F 2 "LED_SMD:LED_0603_1608Metric_Pad1.05x0.95mm_HandSolder" H 4750 4200 50  0001 C CNN
+F 3 "~" H 4750 4200 50  0001 C CNN
+F 4 "150060GS75000" H 4750 4200 50  0001 C CNN "MPN"
+F 5 "Wurth" H 4750 4200 50  0001 C CNN "Mfg"
+	1    4750 4200
+	0    -1   -1   0
+$EndComp
+$Comp
+L Device:LED D1
+U 1 1 5DF6B205
+P 4450 4200
+F 0 "D1" V 4450 4150 50  0000 R CNN
+F 1 "GRN" V 4300 4100 50  0000 R CNN
+F 2 "LED_SMD:LED_0603_1608Metric_Pad1.05x0.95mm_HandSolder" H 4450 4200 50  0001 C CNN
+F 3 "~" H 4450 4200 50  0001 C CNN
+F 4 "150060GS75000" H 4450 4200 50  0001 C CNN "MPN"
+F 5 "Wurth" H 4450 4200 50  0001 C CNN "Mfg"
+	1    4450 4200
+	0    -1   -1   0
+$EndComp
 $EndSCHEMATC
